Commit message: 测试新地图

File: mesh_navigation_tutorials/src/pb_vehicle_adapter/models/pb_navigation_robot.urdf (robot description, URDF)
Before this commit: robot pb_navigation_robot, 10 links, 9 joints
Links:
- link front_left_wheel: geometry collision cylinder length=0.0452 radius=0.0758; visual mesh filename=file:///home/rainple/nav_test_fix/third_party/pb2025_source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
- link front_right_wheel: geometry collision cylinder length=0.0452 radius=0.0758; visual mesh filename=file:///home/rainple/nav_test_fix/third_party/pb2025_source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
- link rear_left_wheel: geometry collision cylinder length=0.0452 radius=0.0758; visual mesh filename=file:///home/rainple/nav_test_fix/third_party/pb2025_source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
- link rear_right_wheel: geometry collision cylinder length=0.0452 radius=0.0758; visual mesh filename=file:///home/rainple/nav_test_fix/third_party/pb2025_source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
